File: lora/lora.kicad_sch (KiCad schematic)
At the start: 22 parts, among them J1 USB_C_Receptacle_USB2.0_14P, J2 Conn_Coaxial, J4 Conn_01x10_Pin, SW1 SW_Push, SW2 SW_Push, U1 ESP32-S3-WROOM-1, U2 SX1262IMLTRT, U3 AMS1117-3.3

Commit message: latest
Parts:
- removed J4: Conn_01x10_Pin, symbol Connector:Conn_01x10_Pin
- added J3, J5: Conn_01x15_Pin, Connector_PinHeader_2.54mm:PinHeader_1x15_P2.54mm_Vertical, symbol Connector:Conn_01x15_Pin
- C1, C2, C3, C4, C5, C6, C7, C8: footprint (none) -> Capacitor_SMD:C_0402_1005Metric
- J1: footprint (none) -> Connector_USB:USB_C_Receptacle_HRO_TYPE-C-31-M-12
- J2: footprint (none) -> Connector_Coaxial:U.FL_Hirose_U.FL-R-SMT-1_Vertical
- L1: footprint (none) -> Inductor_SMD:L_0805_2012Metric
- L2: footprint (none) -> Inductor_SMD:L_0402_1005Metric
- R1, R2, R3, R4: footprint (none) -> Resistor_SMD:R_0402_1005Metric
- SW1, SW2: footprint (none) -> Button_Switch_SMD:SW_SPST_PTS645Sx43SMTR92
Connections:
- net +3V3: now also J3.1 (Pin_1), J3.2 (Pin_2)
- net BUSY: now also J5.13 (Pin_13)
- net DIO1: now also J5.14 (Pin_14)
- net GND: now also J1.SH (SHIELD), J3.3 (Pin_3), J3.4 (Pin_4), J3.5 (Pin_5), J5.15 (Pin_15); no longer J1.S1 (SHIELD)
- net GPIO1: now also J3.12 (Pin_12)
- net GPIO2: now also J3.13 (Pin_13)
- net GPIO47: now also J5.8 (Pin_8)
- net I2C_SCL: now also J3.11 (Pin_11)
- net I2C_SDA: now also J3.10 (Pin_10)
- net SX_RST: now also J5.12 (Pin_12)
- net UART_RX: now also J3.7 (Pin_7)
- net UART_TX: now also J3.6 (Pin_6)
- net USB_DN: now also J3.15 (Pin_15)
- net USB_DP: now also J3.14 (Pin_14)
- net GPS_RX: now reaches U1.10 (IO17)
- net GPS_RX: now also J5.2 (Pin_2)
- net GPIO46: now reaches U1.16 (IO46)
- net GPIO46: now also J5.10 (Pin_10)
- net GPIO48: now reaches U1.25 (IO48)
- net GPIO48: now also J5.11 (Pin_11)
- net GPIO45: now reaches U1.26 (IO45)
- net GPIO45: now also J5.9 (Pin_9)
- net GPIO39: now reaches U1.32 (IO39)
- net GPIO39: now also J5.4 (Pin_4)
- net GPIO40: now reaches U1.33 (IO40)
- net GPIO40: now also J5.5 (Pin_5)
- net GPIO41: now reaches U1.34 (IO41)
- net GPIO41: now also J5.6 (Pin_6)
- net GPIO42: now reaches U1.35 (IO42)
- net GPIO42: now also J5.7 (Pin_7)
- net GPS_PPS: now reaches U1.8 (IO15)
- net GPS_PPS: now also J5.3 (Pin_3)
- net GPS_TX: now reaches U1.9 (IO16)
- net GPS_TX: now also J5.1 (Pin_1)
- new net UART2_RX: J3.9 (Pin_9)
- new net UART2_TX: J3.8 (Pin_8)
- no-connect marks 18 -> 15
Other:
- moved on the sheet: C1, C2, C3, C4, C5, C6, C7, C8, J1, J2, L1, L2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
